Commit message: Your commit message describing the changes

File: src/bumperbot_description/urdf/bumperbot.urdf.xacro (robot description, xacro)
@@ -192,3 +192,33 @@
     <axis xyz="0 0 0" />
   </joint>
+  <joint name="camera_joint" type="fixed">
+    <parent link="base_link"/>
+    <child link="camera_link"/>
+    <origin xyz="0.0 0.0 0.2" rpy="0 0 0"/> <!-- Adjust position of the camera -->
+  </joint>
+  <!-- Camera Link -->
+  <link name="camera_link">
+  <inertial>
+    <origin xyz="0.07 0 -0.15" rpy="0 0 0"/>
+    <mass value="0.2"/>
+    <inertia ixx="8.33e-05" ixy="0" ixz="0"
+             iyy="8.33e-05" iyz="0"
+             izz="8.33e-05"/>
+  </inertial>
+  <visual>
+    <origin xyz="0.07 0 -0.15" rpy="0 0 0"/>
+    <geometry>
+      <box size="0.03 0.03 0.03"/> <!-- Represent the camera visually -->
+    </geometry>
+    <material name="red">
+      <color rgba="1.0 0.0 0.0 1.0"/> <!-- Red color -->
+    </material>
+  </visual>
+  <collision>
+    <origin xyz="0.07 0 -0.15" rpy="0 0 0"/>
+    <geometry>
+      <box size="0.03 0.03 0.03"/>
+    </geometry>
+  </collision>
+</link>
 </robot>

File: src/bumperbot_description/urdf/bumperbot_gazebo.xacro (robot description, xacro)
@@ -101,3 +101,29 @@
   </sensor>
 </gazebo>
+<!-- camera plugin -->
+<gazebo reference="camera_link">
+    <sensor type="camera" name="camera_sensor">
+      <update_rate>30</update_rate>
+      <camera>
+        <horizontal_fov>1.5708</horizontal_fov> <!-- 90 degrees FOV -->
+        <image>
+          <width>640</width>
+          <height>480</height>
+          <format>R8G8B8</format>
+        </image>
+        <clip>
+          <near>0.1</near>
+          <far>100</far>
+        </clip>
+      </camera>
+      <plugin name="camera_controller" filename="libgazebo_ros_camera.so">
+        <alwaysOn>true</alwaysOn>
+        <updateRate>30</updateRate>
+        <cameraName>bumperbot_camera</cameraName>
+        <imageTopicName>/camera/image_raw</imageTopicName>
+        <cameraInfoTopicName>/camera/camera_info</cameraInfoTopicName>
+        <frameName>camera_link</frameName>
+      </plugin>
+    </sensor>
+  </gazebo>
 </robot>
